Commit message: change params

File: src/bot_description/urdf/bot.urdf.xacro (robot description, xacro)
@@ -68,4 +68,17 @@
     <child link="rslidar_link" />
   </joint>
+  <link name="imu_link">
+    <!-- <visual>
+        <origin xyz="0.0 0.0 0.0" />
+        <geometry>
+            <cylinder length="0.05" radius="0.03" />
+        </geometry>
+    </visual> -->
+  </link>
+  <joint name="imu_joint" type="fixed">
+    <origin xyz="0 0 0" rpy="0 0 0" />
+    <parent link="base_link" />
+    <child link="imu_link" />
+  </joint>
   <xacro:scout_wheel wheel_prefix="front_right">
     <origin xyz="${wheelbase/2} ${-wheeltrack/2} ${wheel_vertical_offset}" rpy="${M_PI} 0 0" />
